Commit message: 25/6

File: Assem1.SLDASM/urdf/Assem1.SLDASM.urdf (robot description, URDF)
Before this commit: robot Assem1.SLDASM, 5 links, 4 joints
Links:
- link Left wheel: mass 0.030159 -> 0.087
- link Link1: mass 0.040888 -> 0.087
- link Right Wheel: mass 0.030159 -> 0.05
- link base_link: mass 0.17195 -> 0.15
